File: rp-tkl.kicad_pcb (KiCad board)
At the start: 2 copper layers, 344.7 x 123.1 mm, 235 parts, among them J1 USB_C_Receptacle_USB2.0, J2 SWD, SW0 SW_Push, SW1 ?, SW10 ?, SW100 ?, SW101 ?, SW102 ?, SW103 ?, SW104 ?, SW11 ?, SW12 ?, SW13 ?, SW14 ?, SW15 ?, SW16 ?, SW17 ?, SW18 ?, SW19 ?, SW2 ?, SW20 ?, SW21 ?, SW22 ?, SW23 ?, SW24 ?, SW25 ?, SW26 ?, SW27 ?, SW28 ?, SW29 ?, SW3 ?, SW30 ?, SW31 ?, SW32 ?, SW33 ?, SW34 ?, SW35 ?, SW36 ?, SW37 ?, SW38 ?, SW39 ?, SW4 ?, SW40 ?, SW41 ?, SW42 ?, SW43 ?, SW44 ?, SW45 ?, SW46 ?, SW47 ?, SW48 ?, SW49 ?, SW5 ?, SW50 ?, SW51 ?, SW52 ?, SW53 ?, SW54 ?, SW55 ?, SW56 ?, SW57 ?, SW58 ?, SW59 ?, SW6 ?, SW60 ?, SW61 ?, SW62 ?, SW63 ?, SW64 ?, SW65 ?, SW66 ?, SW67 ?, SW68 ?, SW69 ?, SW7 ?, SW70 ?, SW71 ?, SW72 ?, SW73 ?, SW74 ?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

Commit message: [Preliminary] Matrix routed
Parts:
- moved D85 7.49 mm to (249.6, 162.1), turned to -90 degrees
- moved D49 4.05 mm to (320.3, 117.7)
Routing:
- net ROW1: track 0.00 -> 339.8 mm, vias 0 -> 2
- net ROW5: track 0.00 -> 334.9 mm
- net ROW2: track 0.00 -> 331.1 mm, vias 0 -> 2
- net ROW0: track 0.00 -> 304.8 mm
- net ROW4: track 0.00 -> 302.9 mm
- net ROW3: track 0.00 -> 252.7 mm
- net COL16: track 0.00 -> 189.3 mm
- net COL15: track 0.00 -> 181.9 mm
- net COL12: track 0.00 -> 155.3 mm
- net COL14: track 0.00 -> 144.7 mm
- net COL0: track 0.00 -> 138.0 mm
- net COL6: track 0.00 -> 132.5 mm
- net COL2: track 0.00 -> 132.5 mm
- net COL11: track 0.00 -> 127.3 mm
- net COL10: track 0.00 -> 115.6 mm
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